Commit message: Updated xacros.

File: samples/ahl_pr2_description/urdf/arm/arm.property.xacro (robot description, xacro)
@@ -1,8 +1,8 @@
 <?xml version="1.0"?>
 <robot xmlns:xacro="http://ros.org/wiki/xacro">
-  <property name="PI" value="3.1415926535897931"/>
-  <property name="shoulder_pan_x" value="0.21"/>
-  <property name="shoulder_pan_y" value="0.188"/>
-  <property name="shoulder_pan_z" value="0.195"/>
+  <xacro:property name="PI" value="3.1415926535897931"/>
+  <xacro:property name="shoulder_pan_x" value="0.21"/>
+  <xacro:property name="shoulder_pan_y" value="0.188"/>
+  <xacro:property name="shoulder_pan_z" value="0.195"/>
   <xacro:macro name="shoulder_pan_inertial">
     <inertial>
@@ -12,13 +12,13 @@
     </inertial>
   </xacro:macro>
-  <property name="shoulder_pan_damping" value="10.0"/>
-  <property name="shoulder_pan_friction" value="0"/>
-  <property name="shoulder_pan_effort" value="10000"/>
-  <property name="shoulder_pan_velocity" value="10000"/>
-  <property name="shoulder_pan_upper" value="2.285404"/>
-  <property name="shoulder_pan_lower" value="-0.714602"/>
-  <property name="shoulder_lift_x" value="0.1"/>
-  <property name="shoulder_lift_y" value="0"/>
-  <property name="shoulder_lift_z" value="-0.142"/>
+  <xacro:property name="shoulder_pan_damping" value="10.0"/>
+  <xacro:property name="shoulder_pan_friction" value="0"/>
+  <xacro:property name="shoulder_pan_effort" value="10000"/>
+  <xacro:property name="shoulder_pan_velocity" value="10000"/>
+  <xacro:property name="shoulder_pan_upper" value="2.285404"/>
+  <xacro:property name="shoulder_pan_lower" value="-0.714602"/>
+  <xacro:property name="shoulder_lift_x" value="0.1"/>
+  <xacro:property name="shoulder_lift_y" value="0"/>
+  <xacro:property name="shoulder_lift_z" value="-0.142"/>
   <xacro:macro name="shoulder_lift_inertial">
     <inertial>
@@ -28,13 +28,13 @@
     </inertial>
   </xacro:macro>
-  <property name="shoulder_lift_damping" value="10.0"/>
-  <property name="shoulder_lift_friction" value="0"/>
-  <property name="shoulder_lift_effort" value="10000"/>
-  <property name="shoulder_lift_velocity" value="10000"/>
-  <property name="shoulder_lift_upper" value="1.396300"/>
-  <property name="shoulder_lift_lower" value="-0.523601"/>
-  <property name="upper_arm_x" value="0.12"/>
-  <property name="upper_arm_y" value="0"/>
-  <property name="upper_arm_z" value="0"/>
+  <xacro:property name="shoulder_lift_damping" value="10.0"/>
+  <xacro:property name="shoulder_lift_friction" value="0"/>
+  <xacro:property name="shoulder_lift_effort" value="10000"/>
+  <xacro:property name="shoulder_lift_velocity" value="10000"/>
+  <xacro:property name="shoulder_lift_upper" value="1.396300"/>
+  <xacro:property name="shoulder_lift_lower" value="-0.523601"/>
+  <xacro:property name="upper_arm_x" value="0.12"/>
+  <xacro:property name="upper_arm_y" value="0"/>
+  <xacro:property name="upper_arm_z" value="0"/>
   <xacro:macro name="upper_arm_inertial">
     <inertial>
@@ -44,14 +44,14 @@
     </inertial>
   </xacro:macro>
-  <property name="upper_arm_damping" value="0.1"/>
-  <property name="upper_arm_friction" value="0"/>
-  <property name="upper_arm_effort" value="10000"/>
-  <property name="upper_arm_velocity" value="10000"/>
-  <property name="upper_arm_upper" value="3.900008"/>
-<!--  <property name="upper_arm_lower" value="-0.800000"/> -->
-  <property name="upper_arm_lower" value="-3.900008"/>
-  <property name="elbow_x" value="0.28"/>
-  <property name="elbow_y" value="0"/>
-  <property name="elbow_z" value="0"/>
+  <xacro:property name="upper_arm_damping" value="0.1"/>
+  <xacro:property name="upper_arm_friction" value="0"/>
+  <xacro:property name="upper_arm_effort" value="10000"/>
+  <xacro:property name="upper_arm_velocity" value="10000"/>
+  <xacro:property name="upper_arm_upper" value="3.900008"/>
+<!--  <xacro:property name="upper_arm_lower" value="-0.800000"/> -->
+  <xacro:property name="upper_arm_lower" value="-3.900008"/>
+  <xacro:property name="elbow_x" value="0.28"/>
+  <xacro:property name="elbow_y" value="0"/>
+  <xacro:property name="elbow_z" value="0"/>
   <xacro:macro name="elbow_inertial">
     <inertial>
@@ -61,13 +61,13 @@
     </inertial>
   </xacro:macro>
-  <property name="elbow_damping" value="1.0"/>
-  <property name="elbow_friction" value="0"/>
-  <property name="elbow_effort" value="10000"/>
-  <property name="elbow_velocity" value="10000"/>
-  <property name="elbow_upper" value="1.0"/>
-  <property name="elbow_lower" value="-2.321305"/>
-  <property name="forearm_x" value="0.09"/>
-  <property name="forearm_y" value="0"/>
-  <property name="forearm_z" value="0"/>
+  <xacro:property name="elbow_damping" value="1.0"/>
+  <xacro:property name="elbow_friction" value="0"/>
+  <xacro:property name="elbow_effort" value="10000"/>
+  <xacro:property name="elbow_velocity" value="10000"/>
+  <xacro:property name="elbow_upper" value="1.0"/>
+  <xacro:property name="elbow_lower" value="-2.321305"/>
+  <xacro:property name="forearm_x" value="0.09"/>
+  <xacro:property name="forearm_y" value="0"/>
+  <xacro:property name="forearm_z" value="0"/>
   <xacro:macro name="forearm_inertial">
     <inertial>
@@ -77,13 +77,13 @@
     </inertial>
   </xacro:macro>
-  <property name="forearm_damping" value="0.1"/>
-  <property name="forearm_friction" value="0"/>
-  <property name="forearm_effort" value="10000"/>
-  <property name="forearm_velocity" value="10000"/>
-  <property name="forearm_upper" value="10000000"/>
-  <property name="forearm_lower" value="-10000000"/>
-  <property name="wrist_flex_x" value="0.23"/>
-  <property name="wrist_flex_y" value="0"/>
-  <property name="wrist_flex_z" value="0"/>
+  <xacro:property name="forearm_damping" value="0.1"/>
+  <xacro:property name="forearm_friction" value="0"/>
+  <xacro:property name="forearm_effort" value="10000"/>
+  <xacro:property name="forearm_velocity" value="10000"/>
+  <xacro:property name="forearm_upper" value="10000000"/>
+  <xacro:property name="forearm_lower" value="-10000000"/>
+  <xacro:property name="wrist_flex_x" value="0.23"/>
+  <xacro:property name="wrist_flex_y" value="0"/>
+  <xacro:property name="wrist_flex_z" value="0"/>
   <xacro:macro name="wrist_flex_inertial">
     <inertial>
@@ -93,13 +93,13 @@
     </inertial>
   </xacro:macro>
-  <property name="wrist_flex_damping" value="0.1"/>
-  <property name="wrist_flex_friction" value="0"/>
-  <property name="wrist_flex_effort" value="10000"/>
-  <property name="wrist_flex_velocity" value="10000"/>
-  <property name="wrist_flex_upper" value="1.0"/>
-  <property name="wrist_flex_lower" value="-2.180004"/>
-  <property name="wrist_roll_x" value="0.03"/>
-  <property name="wrist_roll_y" value="0"/>
-  <property name="wrist_roll_z" value="0"/>
+  <xacro:property name="wrist_flex_damping" value="0.1"/>
+  <xacro:property name="wrist_flex_friction" value="0"/>
+  <xacro:property name="wrist_flex_effort" value="10000"/>
+  <xacro:property name="wrist_flex_velocity" value="10000"/>
+  <xacro:property name="wrist_flex_upper" value="1.0"/>
+  <xacro:property name="wrist_flex_lower" value="-2.180004"/>
+  <xacro:property name="wrist_roll_x" value="0.03"/>
+  <xacro:property name="wrist_roll_y" value="0"/>
+  <xacro:property name="wrist_roll_z" value="0"/>
   <xacro:macro name="wrist_roll_inertial">
     <inertial>
@@ -109,10 +109,10 @@
     </inertial>
   </xacro:macro>
-  <property name="wrist_roll_damping" value="0.1"/>
-  <property name="wrist_roll_friction" value="0"/>
-  <property name="wrist_roll_effort" value="10000"/>
-  <property name="wrist_roll_velocity" value="10000"/>
-  <property name="wrist_roll_upper" value="10000000"/>
-  <property name="wrist_roll_lower" value="-10000000"/>
+  <xacro:property name="wrist_roll_damping" value="0.1"/>
+  <xacro:property name="wrist_roll_friction" value="0"/>
+  <xacro:property name="wrist_roll_effort" value="10000"/>
+  <xacro:property name="wrist_roll_velocity" value="10000"/>
+  <xacro:property name="wrist_roll_upper" value="10000000"/>
+  <xacro:property name="wrist_roll_lower" value="-10000000"/>
   <xacro:macro name="gripper_joint_origin">
     <origin xyz="0.088 0 0" rpy="0 0 0"/>

File: samples/ahl_pr2_description/urdf/base/base.property.xacro (robot description, xacro)
@@ -1,5 +1,5 @@
 <?xml version="1.0"?>
 <robot xmlns:xacro="http://ros.org/wiki/xacro">
-  <property name="M_PI" value="3.1415926535897931"/>
+  <xacro:property name="M_PI" value="3.1415926535897931"/>
   <xacro:macro name="base_x_inertial">
     <inertial>
@@ -17,10 +17,10 @@
     </visual>
   </xacro:macro>
-  <property name="base_x_damping" value="10"/>
-  <property name="base_x_friction" value="0.2"/>
-  <property name="base_x_effort" value="10000"/>
-  <property name="base_x_velocity" value="10000"/>
-  <property name="base_x_upper" value="1000000"/>
-  <property name="base_x_lower" value="-1000000"/>
+  <xacro:property name="base_x_damping" value="10"/>
+  <xacro:property name="base_x_friction" value="0.2"/>
+  <xacro:property name="base_x_effort" value="10000"/>
+  <xacro:property name="base_x_velocity" value="10000"/>
+  <xacro:property name="base_x_upper" value="1000000"/>
+  <xacro:property name="base_x_lower" value="-1000000"/>
   <xacro:macro name="base_y_inertial">
     <inertial>
@@ -38,10 +38,10 @@
     </visual>
   </xacro:macro>
-  <property name="base_y_damping" value="10"/>
-  <property name="base_y_friction" value="0.2"/>
-  <property name="base_y_effort" value="10000"/>
-  <property name="base_y_velocity" value="10000"/>
-  <property name="base_y_upper" value="1000000"/>
-  <property name="base_y_lower" value="-1000000"/>
+  <xacro:property name="base_y_damping" value="10"/>
+  <xacro:property name="base_y_friction" value="0.2"/>
+  <xacro:property name="base_y_effort" value="10000"/>
+  <xacro:property name="base_y_velocity" value="10000"/>
+  <xacro:property name="base_y_upper" value="1000000"/>
+  <xacro:property name="base_y_lower" value="-1000000"/>
   <xacro:macro name="base_yaw_inertial">
     <inertial>
@@ -59,10 +59,10 @@
     </visual>
   </xacro:macro>
-  <property name="base_yaw_damping" value="10"/>
-  <property name="base_yaw_friction" value="0.2"/>
-  <property name="base_yaw_effort" value="10000"/>
-  <property name="base_yaw_velocity" value="10000"/>
-  <property name="base_yaw_upper" value="1000000"/>
-  <property name="base_yaw_lower" value="-1000000"/>
+  <xacro:property name="base_yaw_damping" value="10"/>
+  <xacro:property name="base_yaw_friction" value="0.2"/>
+  <xacro:property name="base_yaw_effort" value="10000"/>
+  <xacro:property name="base_yaw_velocity" value="10000"/>
+  <xacro:property name="base_yaw_upper" value="1000000"/>
+  <xacro:property name="base_yaw_lower" value="-1000000"/>
   <xacro:macro name="base_link_inertial">
     <inertial>
@@ -72,7 +72,7 @@
     </inertial>
   </xacro:macro>
-  <property name="caster_x" value="0.218"/>
-  <property name="caster_y" value="0.218"/>
-  <property name="caster_z" value="0.2"/>
+  <xacro:property name="caster_x" value="0.218"/>
+  <xacro:property name="caster_y" value="0.218"/>
+  <xacro:property name="caster_z" value="0.2"/>
   <xacro:macro name="caster_inertial">
     <inertial>
@@ -93,11 +93,11 @@
     </visual>
   </xacro:macro>
-  <property name="caster_damping" value="0.7"/>
-  <property name="caster_friction" value="0.2"/>
-  <property name="caster_effort" value="10000"/>
-  <property name="caster_velocity" value="10000"/>
-  <property name="caster_upper" value="1000000"/>
-  <property name="caster_lower" value="-1000000"/>
-  <property name="wheel_z" value="-0.17"/>
+  <xacro:property name="caster_damping" value="0.7"/>
+  <xacro:property name="caster_friction" value="0.2"/>
+  <xacro:property name="caster_effort" value="10000"/>
+  <xacro:property name="caster_velocity" value="10000"/>
+  <xacro:property name="caster_upper" value="1000000"/>
+  <xacro:property name="caster_lower" value="-1000000"/>
+  <xacro:property name="wheel_z" value="-0.17"/>
   <xacro:macro name="wheel_inertial">
     <inertial>
@@ -107,15 +107,15 @@
     </inertial>
   </xacro:macro>
-  <property name="wheel_radius" value="0.075"/>
-  <property name="wheel_length" value="0.10"/>
-  <property name="wheel_damping" value="0.7"/>
-  <property name="wheel_friction" value="0.2"/>
-  <property name="wheel_effort" value="10000"/>
-  <property name="wheel_velocity" value="10000"/>
-  <property name="wheel_upper" value="1000000"/>
-  <property name="wheel_lower" value="-1000000"/>
-  <property name="torso_x" value="-0.255"/>
-  <property name="torso_y" value="0"/>
-  <property name="torso_z" value="0.66"/>
+  <xacro:property name="wheel_radius" value="0.075"/>
+  <xacro:property name="wheel_length" value="0.10"/>
+  <xacro:property name="wheel_damping" value="0.7"/>
+  <xacro:property name="wheel_friction" value="0.2"/>
+  <xacro:property name="wheel_effort" value="10000"/>
+  <xacro:property name="wheel_velocity" value="10000"/>
+  <xacro:property name="wheel_upper" value="1000000"/>
+  <xacro:property name="wheel_lower" value="-1000000"/>
+  <xacro:property name="torso_x" value="-0.255"/>
+  <xacro:property name="torso_y" value="0"/>
+  <xacro:property name="torso_z" value="0.66"/>
   <xacro:macro name="torso_inertial">
     <inertial>
@@ -125,9 +125,9 @@
     </inertial>
   </xacro:macro>
-  <property name="torso_damping" value="30.0"/>
-  <property name="torso_friction" value="0.1"/>
-  <property name="torso_effort" value="10000"/>
-  <property name="torso_velocity" value="4.0"/>
-  <property name="torso_upper" value="0.33"/>
-  <property name="torso_lower" value="0"/>
+  <xacro:property name="torso_damping" value="30.0"/>
+  <xacro:property name="torso_friction" value="0.1"/>
+  <xacro:property name="torso_effort" value="10000"/>
+  <xacro:property name="torso_velocity" value="4.0"/>
+  <xacro:property name="torso_upper" value="0.33"/>
+  <xacro:property name="torso_lower" value="0"/>
 </robot>

File: samples/ahl_pr2_description/urdf/gripper/gripper.property.xacro (robot description, xacro)
@@ -1,8 +1,8 @@
 <?xml version="1.0"?>
 <robot xmlns:xacro="http://ros.org/wiki/xacro">
-  <property name="PI" value="3.1415926535897931"/>
-  <property name="finger_x" value="0.0475"/>
-  <property name="finger_y" value="0.01"/>
-  <property name="finger_z" value="0"/>
+  <xacro:property name="PI" value="3.1415926535897931"/>
+  <xacro:property name="finger_x" value="0.0475"/>
+  <xacro:property name="finger_y" value="0.01"/>
+  <xacro:property name="finger_z" value="0"/>
   <xacro:macro name="finger_inertial">
     <inertial>
@@ -12,13 +12,13 @@
     </inertial>
   </xacro:macro>
-  <property name="finger_damping" value="0.1"/>
-  <property name="finger_friction" value="0.7"/>
-  <property name="finger_effort" value="10000"/>
-  <property name="finger_velocity" value="0.1"/>
-  <property name="finger_upper" value="0.548"/>
-  <property name="finger_lower" value="0"/>
-  <property name="finger_tip_x" value="0.091"/>
-  <property name="finger_tip_y" value="0.005"/>
-  <property name="finger_tip_z" value="0"/>
+  <xacro:property name="finger_damping" value="0.1"/>
+  <xacro:property name="finger_friction" value="0.7"/>
+  <xacro:property name="finger_effort" value="10000"/>
+  <xacro:property name="finger_velocity" value="0.1"/>
+  <xacro:property name="finger_upper" value="0.548"/>
+  <xacro:property name="finger_lower" value="0"/>
+  <xacro:property name="finger_tip_x" value="0.091"/>
+  <xacro:property name="finger_tip_y" value="0.005"/>
+  <xacro:property name="finger_tip_z" value="0"/>
   <xacro:macro name="finger_tip_inertial">
     <inertial>
@@ -28,9 +28,9 @@
     </inertial>
   </xacro:macro>
-  <property name="finger_tip_damping" value="0.1"/>
-  <property name="finger_tip_friction" value="0.7"/>
-  <property name="finger_tip_effort" value="10000"/>
-  <property name="finger_tip_velocity" value="0.1"/>
-  <property name="finger_tip_upper" value="0.548"/>
-  <property name="finger_tip_lower" value="0"/>
+  <xacro:property name="finger_tip_damping" value="0.1"/>
+  <xacro:property name="finger_tip_friction" value="0.7"/>
+  <xacro:property name="finger_tip_effort" value="10000"/>
+  <xacro:property name="finger_tip_velocity" value="0.1"/>
+  <xacro:property name="finger_tip_upper" value="0.548"/>
+  <xacro:property name="finger_tip_lower" value="0"/>
 </robot>

File: samples/ahl_pr2_description/urdf/head/head.property.xacro (robot description, xacro)
@@ -1,8 +1,8 @@
 <?xml version="1.0"?>
 <robot xmlns:xacro="http://ros.org/wiki/xacro">
-  <property name="PI" value="3.1415926535897931"/>
-  <property name="tilting_hokuyo_x" value="0.31"/>
-  <property name="tilting_hokuyo_y" value="0"/>
-  <property name="tilting_hokuyo_z" value="0.272"/>
+  <xacro:property name="PI" value="3.1415926535897931"/>
+  <xacro:property name="tilting_hokuyo_x" value="0.31"/>
+  <xacro:property name="tilting_hokuyo_y" value="0"/>
+  <xacro:property name="tilting_hokuyo_z" value="0.272"/>
   <xacro:macro name="tilting_hokuyo_inertial">
     <inertial>
@@ -12,13 +12,13 @@
     </inertial>
   </xacro:macro>
-  <property name="tilting_hokuyo_damping" value="1"/>
-  <property name="tilting_hokuyo_friction" value="0"/>
-  <property name="tilting_hokuyo_effort" value="10000"/>
-  <property name="tilting_hokuyo_velocity" value="10000"/>
-  <property name="tilting_hokuyo_upper" value="${M_PI / 2}"/>
-  <property name="tilting_hokuyo_lower" value="${-M_PI / 2}"/>
-  <property name="head_pan_x" value="0.2"/>
-  <property name="head_pan_y" value="0"/>
-  <property name="head_pan_z" value="0.36"/>
+  <xacro:property name="tilting_hokuyo_damping" value="1"/>
+  <xacro:property name="tilting_hokuyo_friction" value="0"/>
+  <xacro:property name="tilting_hokuyo_effort" value="10000"/>
+  <xacro:property name="tilting_hokuyo_velocity" value="10000"/>
+  <xacro:property name="tilting_hokuyo_upper" value="${M_PI / 2}"/>
+  <xacro:property name="tilting_hokuyo_lower" value="${-M_PI / 2}"/>
+  <xacro:property name="head_pan_x" value="0.2"/>
+  <xacro:property name="head_pan_y" value="0"/>
+  <xacro:property name="head_pan_z" value="0.36"/>
   <xacro:macro name="head_pan_inertial">
     <inertial>
@@ -28,13 +28,13 @@
     </inertial>
   </xacro:macro>
-  <property name="head_pan_damping" value="1"/>
-  <property name="head_pan_friction" value="0"/>
-  <property name="head_pan_effort" value="10000"/>
-  <property name="head_pan_velocity" value="10000"/>
-  <property name="head_pan_upper" value="${M_PI / 2}"/>
-  <property name="head_pan_lower" value="${-M_PI / 2}"/>
-  <property name="head_tilt_x" value="0.062"/>
-  <property name="head_tilt_y" value="0"/>
-  <property name="head_tilt_z" value="0.065"/>
+  <xacro:property name="head_pan_damping" value="1"/>
+  <xacro:property name="head_pan_friction" value="0"/>
+  <xacro:property name="head_pan_effort" value="10000"/>
+  <xacro:property name="head_pan_velocity" value="10000"/>
+  <xacro:property name="head_pan_upper" value="${M_PI / 2}"/>
+  <xacro:property name="head_pan_lower" value="${-M_PI / 2}"/>
+  <xacro:property name="head_tilt_x" value="0.062"/>
+  <xacro:property name="head_tilt_y" value="0"/>
+  <xacro:property name="head_tilt_z" value="0.065"/>
   <xacro:macro name="head_tilt_inertial">
     <inertial>
@@ -44,9 +44,9 @@
     </inertial>
   </xacro:macro>
-  <property name="head_tilt_damping" value="1"/>
-  <property name="head_tilt_friction" value="0"/>
-  <property name="head_tilt_effort" value="10000"/>
-  <property name="head_tilt_velocity" value="10000"/>
-  <property name="head_tilt_upper" value="${M_PI / 2}"/>
-  <property name="head_tilt_lower" value="${-M_PI / 2}"/>
+  <xacro:property name="head_tilt_damping" value="1"/>
+  <xacro:property name="head_tilt_friction" value="0"/>
+  <xacro:property name="head_tilt_effort" value="10000"/>
+  <xacro:property name="head_tilt_velocity" value="10000"/>
+  <xacro:property name="head_tilt_upper" value="${M_PI / 2}"/>
+  <xacro:property name="head_tilt_lower" value="${-M_PI / 2}"/>
 </robot>
