Commit message: Modified xacro files to adjust newer version.

File: samples/ahl_youbot_description/urdf/arm/arm.property.xacro (robot description, xacro)
@@ -1,24 +1,24 @@
 <?xml version="1.0"?>
-<robot xmlns:xacro="http://ros.org/wiki/xacro">>
+<robot xmlns:xacro="http://ros.org/wiki/xacro">
   <!-- common properties -->
-  <property name="M_PI" value="3.14159265358979323846"/>
-  <property name="threshold" value="0.01"/>
+  <xacro:property name="M_PI" value="3.14159265358979323846"/>
+  <xacro:property name="threshold" value="0.01"/>
   <!-- arm limits positions (deg) -->
-  <property name="joint1_lower_limit" value="-${M_PI * 169 / 180}"/>
-  <property name="joint1_upper_limit" value= "${M_PI * 169 / 180}"/>
-  <property name="joint2_lower_limit" value="-${M_PI *  65 / 180}"/>
-  <property name="joint2_upper_limit" value= "${M_PI *  90 / 180}"/>
-  <property name="joint3_lower_limit" value="-${M_PI * 151 / 180}"/>
-  <property name="joint3_upper_limit" value= "${M_PI * 146 / 180}"/>
-  <property name="joint4_lower_limit" value="-${M_PI * 102.5 / 180}"/>
-  <property name="joint4_upper_limit" value= "${M_PI * 102.5 / 180}"/>
-  <property name="joint5_lower_limit" value="-${M_PI * 165 / 180}"/>
-  <property name="joint5_upper_limit" value= "${M_PI * 165 / 180}"/>
+  <xacro:property name="joint1_lower_limit" value="-${M_PI * 169 / 180}"/>
+  <xacro:property name="joint1_upper_limit" value= "${M_PI * 169 / 180}"/>
+  <xacro:property name="joint2_lower_limit" value="-${M_PI *  65 / 180}"/>
+  <xacro:property name="joint2_upper_limit" value= "${M_PI *  90 / 180}"/>
+  <xacro:property name="joint3_lower_limit" value="-${M_PI * 151 / 180}"/>
+  <xacro:property name="joint3_upper_limit" value= "${M_PI * 146 / 180}"/>
+  <xacro:property name="joint4_lower_limit" value="-${M_PI * 102.5 / 180}"/>
+  <xacro:property name="joint4_upper_limit" value= "${M_PI * 102.5 / 180}"/>
+  <xacro:property name="joint5_lower_limit" value="-${M_PI * 165 / 180}"/>
+  <xacro:property name="joint5_upper_limit" value= "${M_PI * 165 / 180}"/>
   <!-- dynamic properties : mass (kg) Alu data sheet -->
-  <property name="link1_mass" value="1.390"/>
-  <property name="link2_mass" value="1.318"/>
-  <property name="link3_mass" value="0.821"/>
-  <property name="link4_mass" value="0.769"/>
-  <property name="link5_mass" value="0.906"/>
+  <xacro:property name="link1_mass" value="1.390"/>
+  <xacro:property name="link2_mass" value="1.318"/>
+  <xacro:property name="link3_mass" value="0.821"/>
+  <xacro:property name="link4_mass" value="0.769"/>
+  <xacro:property name="link5_mass" value="0.906"/>
   <xacro:macro name="link1_inertia_tensor">
     <origin xyz="-0.010838 0.006337 0.034345" rpy="0 0 0"/>

File: samples/ahl_youbot_description/urdf/base/base.transmission.xacro (robot description, xacro)
@@ -4,6 +4,6 @@
        xmlns:interface="http://playerstage.sourceforge.net/gazebo/xmlschema/#interface"
        xmlns:xacro="http://ros.org/wiki/xacro">
-<!--  <property name="wheel_mechanical_reduction" value="${624/35 * 80/18}"/> -->
-  <property name="wheel_mechanical_reduction" value="1"/>
+<!--  <xacro:property name="wheel_mechanical_reduction" value="${624/35 * 80/18}"/> -->
+  <xacro:property name="wheel_mechanical_reduction" value="1"/>
   <xacro:macro name="youbot_base_transmission">
     <transmission name="base_x_trans">
